File: modules/power_linear_sot_223_1117_5_v_output/working/kicad/current_version/working/working.kicad_sch (KiCad schematic)
At the start: 3 parts, among them J1 pms2231117

Commit message: gitignore update mainly and update
Parts:
- removed C1, C2: catuf4d7, oomlout_oomp_part_footprints:catuf4d7_electronic_capacitor_3216_avx_a_tantalum_4_7_micro_farad_16_volt, symbol oomlout_oomp_part_symbols:catuf4d7_electronic_capacitor_3216_avx_a_tantalum_4_7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
- removed J1: pms2231117, pms2231117_electronic_pmic_sot_223_linear_1117_5v, symbol oomlout_oomp_part_symbols:pms2231117_electronic_pmic_sot_223_linear_1117_5v
- added C1, C2: catuf4d716v, catuf4d716v_electronic_capacitor_3216_avx_a_tantalum_4_7_micro_farad_16_volt, symbol oomlout_oomp_part_symbols:catuf4d716v_electronic_capacitor_3216_avx_a_tantalum_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
- added J?: pms22311171d5v, pms22311171d5v_electronic_pmic_sot_223_linear_1117_1_5_volt, symbol oomlout_oomp_part_symbols:pms22311171d5v_electronic_pmic_sot_223_linear_1117_1_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
Connections:
- net +12V: now also C2.1, J?.3 (VI)
- net GND: now also C1.2, C2.2, J?.1 (GND)
- new net +5V: C1.1, J?.2 (VO)
Other:
- note added: "name"
- note added: "oomp power linear sot223 1117 5_volt"
- note added: "power_5v"
- note removed: "module power linear sot_223 1117 5_v_output"
Changed lines of the file:
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@@
   (junction (at 125.73 99.06) (diameter 0) (color 0 0 0 0)
   )
+  (junction (at 153.67 99.06) (diameter 0) (color 0 0 0 0)
+  )
   (junction (at 139.7 109.22) (diameter 0) (color 0 0 0 0)
-  )
-  (junction (at 153.67 99.06) (diameter 0) (color 0 0 0 0)
   )
   (wire (pts (xy 139.7 109.22) (xy 125.73 109.22))
@@
     (fill (type none))
   )
-  (text "module\npower\nlinear\nsot_223\n1117\n5_v_output\n" (at 109.22 81.28 0)
+  (rectangle (start 133.35 55.88) (end 171.45 62.23)
+    (stroke (width 1) (type default))
+    (fill (type color) (color 0 0 0 0))
+  )
+  (text "oomp\npower\nlinear\nsot223\n1117\n5_volt" (at 109.22 80.01 0)
     (effects (font (size 2.5 2.5)) (justify left bottom))
+  )
+  (text "name" (at 135.89 62.23 90)
+    (effects (font (size 1.27 1.27) (thickness 0.254) bold (color 255 255 255 1)) (justify left bottom))
+  )
+  (text "power_5v\n" (at 170.18 62.23 0)
+    (effects (font (size 4 4) (thickness 0.8) bold (color 255 255 255 1)) (justify right bottom))
   )
   (label "vin" (at 121.92 92.71 90) (fields_autoplaced)
     (effects (font (size 1.27 1.27)) (justify left bottom))
   )
-  (symbol (lib_id "oomlout_oomp_part_symbols:catuf4d7_electronic_capacitor_3216_avx_a_tantalum_4_7_micro_farad_16_volt") (at 153.67 102.87 0) (unit 1)
+  (symbol (lib_id "power:+5V") (at 153.67 92.71 0) (unit 1)
+    (in_bom yes) (on_board yes) (dnp no) (fields_autoplaced)
+    (property "Reference" "#PWR01" (at 153.67 96.52 0)
+      (effects (font (size 1.27 1.27)) hide)
+    )
+    (property "Value" "+5V" (at 153.67 87.63 0)
+      (effects (font (size 1.27 1.27)))
+    )
+    (property "Footprint" "" (at 153.67 92.71 0)
+      (effects (font (size 1.27 1.27)) hide)
+    )
+    (property "Datasheet" "" (at 153.67 92.71 0)
+      (effects (font (size 1.27 1.27)) hide)
+    )
+    (pin "1")
+    (instances
+      (project "working"
+        (path "/b2804c28-0f7b-4aef-9942-b5794639a3dd"
+          (reference "#PWR01") (unit 1)
+        )
+      )
+    )
+  )
+  (symbol (lib_id "oomlout_oomp_part_symbols:pms22311171d5v_electronic_pmic_sot_223_linear_1117_1_5_volt") (at 139.7 99.06 0) (unit 1)
+    (in_bom yes) (on_board yes) (dnp no) (fields_autoplaced)
+    (property "Reference" "J?" (at 139.7 92.71 0)
+      (effects (font (size 1.27 1.27)))
+    )
+    (property "Value" "pms22311171d5v" (at 139.7 95.25 0)
+      (effects (font (size 1.27 1.27)))
+    )
+    (property "Footprint" "pms22311171d5v_electronic_pmic_sot_223_linear_1117_1_5_volt" (at 139.7 93.98 0)
+      (effects (font (size 1.27 1.27)) hide)
+    )
+    (property "Datasheet" "https://github.com/oomlout/oomlout_oomp_v3/parts/electronic_pmic_sot_223_linear_1117_1_5_volt/datasheet.pdf" (at 142.24 105.41 0)
+      (effects (font (size 1.27 1.27)) hide)
+    )
+    (pin "1")
+    (pin "2")
+    (pin "3")
+    (instances
+      (project "working"
+        (path "/b2804c28-0f7b-4aef-9942-b5794639a3dd"
+          (reference "J?") (unit 1)
+        )
+      )
+    )
+  )
+  (symbol (lib_id "oomlout_oomp_part_symbols:catuf4d716v_electronic_capacitor_3216_avx_a_tantalum_4_7_micro_farad_16_volt") (at 125.73 102.87 0) (mirror y) (unit 1)
     (in_bom yes) (on_board yes) (dnp no)
-    (property "Reference" "C2" (at 157.48 100.711 0)
-      (effects (font (size 1.27 1.27)) (justify left))
-    )
-    (property "Value" "catuf4d7" (at 162.56 107.95 90)
-      (effects (font (size 1.27 1.27)) (justify left))
-    )
-    (property "Footprint" "oomlout_oomp_part_footprints:catuf4d7_electronic_capacitor_3216_avx_a_tantalum_4_7_micro_farad_16_volt" (at 154.6352 106.68 0)
-      (effects (font (size 1.27 1.27)) hide)
-    )
-    (property "Datasheet" "https://github.com/oomlout/oomlout_oomp_v3/parts/electronic_capacitor_3216_avx_a_tantalum_4_7_micro_farad_16_volt/datasheet.pdf" (at 153.67 102.87 0)
+    (property "Reference" "C2" (at 132.08 102.87 0)
+      (effects (font (size 1.27 1.27)) (justify left))
+    )
+    (property "Value" "catuf4d716v" (at 120.65 109.22 90)
+      (effects (font (size 1.27 1.27)) (justify left))
+    )
+    (property "Footprint" "catuf4d716v_electronic_capacitor_3216_avx_a_tantalum_4_7_micro_farad_16_volt" (at 124.7648 106.68 0)
+      (effects (font (size 1.27 1.27)) hide)
+    )
+    (property "Datasheet" "https://github.com/oomlout/oomlout_oomp_v3/parts/electronic_capacitor_3216_avx_a_tantalum_4_7_micro_farad_16_volt/datasheet.pdf" (at 125.73 102.87 0)
       (effects (font (size 1.27 1.27)) hide)
     )
@@
     (instances
       (project "working"
-        (path "/917ab96c-dc02-4c3c-8b08-e7587cff047e"
+        (path "/b2804c28-0f7b-4aef-9942-b5794639a3dd"
           (reference "C2") (unit 1)
-        )
-      )
-      (project "working"
-        (path "/b2804c28-0f7b-4aef-9942-b5794639a3dd"
-          (reference "C2") (unit 1)
-        )
-      )
-    )
-  )
-  (symbol (lib_id "oomlout_oomp_part_symbols:catuf4d7_electronic_capacitor_3216_avx_a_tantalum_4_7_micro_farad_16_volt") (at 125.73 102.87 0) (unit 1)
-    (in_bom yes) (on_board yes) (dnp no)
-    (property "Reference" "C1" (at 129.54 100.711 0)
-      (effects (font (size 1.27 1.27)) (justify left))
-    )
-    (property "Value" "catuf4d7" (at 120.65 107.95 90)
-      (effects (font (size 1.27 1.27)) (justify left))
-    )
-    (property "Footprint" "oomlout_oomp_part_footprints:catuf4d7_electronic_capacitor_3216_avx_a_tantalum_4_7_micro_farad_16_volt" (at 126.6952 106.68 0)
-      (effects (font (size 1.27 1.27)) hide)
-    )
-    (property "Datasheet" "https://github.com/oomlout/oomlout_oomp_v3/parts/electronic_capacitor_3216_avx_a_tantalum_4_7_micro_farad_16_volt/datasheet.pdf" (at 125.73 102.87 0)
-      (effects (font (size 1.27 1.27)) hide)
-    )
-    (pin "1")
-    (pin "2")
-    (instances
-      (project "working"
-        (path "/917ab96c-dc02-4c3c-8b08-e7587cff047e"
-          (reference "C1") (unit 1)
-        )
-      )
-      (project "working"
-        (path "/b2804c28-0f7b-4aef-9942-b5794639a3dd"
-          (reference "C1") (unit 1)
         )
       )
@@
       (project "working"
         (path "/b2804c28-0f7b-4aef-9942-b5794639a3dd"
-          (reference "#PWR01") (unit 1)
+          (reference "#PWR?") (unit 1)
+        )
+      )
+    )
+  )
+  (symbol (lib_id "oomlout_oomp_part_symbols:catuf4d716v_electronic_capacitor_3216_avx_a_tantalum_4_7_micro_farad_16_volt") (at 153.67 102.87 0) (unit 1)
+    (in_bom yes) (on_board yes) (dnp no)
+    (property "Reference" "C1" (at 147.32 102.87 0)
+      (effects (font (size 1.27 1.27)) (justify left))
+    )
+    (property "Value" "catuf4d716v" (at 158.75 109.22 90)
+      (effects (font (size 1.27 1.27)) (justify left))
+    )
+    (property "Footprint" "catuf4d716v_electronic_capacitor_3216_avx_a_tantalum_4_7_micro_farad_16_volt" (at 154.6352 106.68 0)
+      (effects (font (size 1.27 1.27)) hide)
+    )
+    (property "Datasheet" "https://github.com/oomlout/oomlout_oomp_v3/parts/electronic_capacitor_3216_avx_a_tantalum_4_7_micro_farad_16_volt/datasheet.pdf" (at 153.67 102.87 0)
+      (effects (font (size 1.27 1.27)) hide)
+    )
+    (pin "1")
+    (pin "2")
+    (instances
+      (project "working"
+        (path "/b2804c28-0f7b-4aef-9942-b5794639a3dd"
+          (reference "C1") (unit 1)
         )
       )
@@
       (project "working"
         (path "/b2804c28-0f7b-4aef-9942-b5794639a3dd"
-          (reference "#PWR02") (unit 1)
-        )
-      )
-    )
-  )
-  (symbol (lib_id "oomlout_oomp_part_symbols:pms2231117_electronic_pmic_sot_223_linear_1117_5v") (at 139.7 99.06 0) (unit 1)
-    (in_bom yes) (on_board yes) (dnp no) (fields_autoplaced)
-    (property "Reference" "J1" (at 139.7 92.71 0)
-      (effects (font (size 1.27 1.27)))
-    )
-    (property "Value" "pms2231117" (at 139.7 95.25 0)
-      (effects (font (size 1.27 1.27)))
-    )
-    (property "Footprint" "pms2231117_electronic_pmic_sot_223_linear_1117_5v" (at 139.7 93.98 0)
-      (effects (font (size 1.27 1.27)) hide)
-    )
-    (property "Datasheet" "https://github.com/oomlout/oomlout_oomp_v3/parts/electronic_pmic_sot_223_linear_1117_5v/datasheet.pdf" (at 142.24 105.41 0)
-      (effects (font (size 1.27 1.27)) hide)
-    )
-    (pin "1")
-    (pin "2")
-    (pin "3")
-    (instances
-      (project "working"
-        (path "/b2804c28-0f7b-4aef-9942-b5794639a3dd"
-          (reference "J1") (unit 1)
-        )
-      )
-    )
-  )
-  (symbol (lib_id "power:+3V3") (at 153.67 92.71 0) (unit 1)
-    (in_bom yes) (on_board yes) (dnp no) (fields_autoplaced)
-    (property "Reference" "#PWR02" (at 153.67 96.52 0)
-      (effects (font (size 1.27 1.27)) hide)
-    )
-    (property "Value" "+3V3" (at 153.67 87.63 0)
-      (effects (font (size 1.27 1.27)))
-    )
-    (property "Footprint" "" (at 153.67 92.71 0)
-      (effects (font (size 1.27 1.27)) hide)
-    )
-    (property "Datasheet" "" (at 153.67 92.71 0)
-      (effects (font (size 1.27 1.27)) hide)
-    )
-    (pin "1")
-    (instances
-      (project "working"
-        (path "/917ab96c-dc02-4c3c-8b08-e7587cff047e"
-          (reference "#PWR02") (unit 1)
-        )
-      )
-      (project "working"
-        (path "/b2804c28-0f7b-4aef-9942-b5794639a3dd"
-          (reference "#PWR03") (unit 1)
-        )
-      )
+          (reference "#PWR?") (unit 1)
+        )
+      )
